File: hardware/teclas.sch (KiCad schematic (older format))
At the start: 20 parts

Commit message: add firmware
Parts:
- C1, C2, C3, C4, C5, C6: renamed from C?; footprint (none) -> Capacitor_SMD:C_0201_0603Metric
- J1: renamed from J?; footprint (none) -> Connector_USB:USB_B_TE_5787834_Vertical
- R1, R2, R3, R4: renamed from R?; footprint (none) -> Resistor_SMD:R_0201_0603Metric
- SW1, SW2, SW3, SW4, SW5, SW6, SW7: renamed from SW?; footprint (none) -> Button_Switch_Keyboard:SW_Cherry_MX_1.00u_PCB
- X1: renamed from X?; footprint (none) -> xtal:XTAL3215; symbol XTAL:XTAL -> teclas-rescue:XTAL-XTAL
- gave numbers to parts that had none: 1
