File: hardware/chiavi.sch (KiCad schematic (older format))
At the start: 20 parts, among them J1 USB_B, SW1 SW_Push, SW2 SW_SPST, SW3 SW_SPST, SW4 SW_SPST, SW5 SW_SPST, SW6 SW_SPST, SW7 SW_SPST, U1 ATmega32U2-AU, X1 XTAL

Commit message: update logo material
Parts:
- X1: symbol teclas-rescue:XTAL-XTAL -> chiavi-rescue:XTAL-XTAL-teclas-rescue
Changed lines of the file:
@@
 encoding utf-8
 Sheet 1 1
-Title "teclas breakdown"
+Title "chiavi breakdown"
 Date "2020-05-10"
 Rev "1.0"
@@
 $EndComp
 $Comp
-L teclas-rescue:XTAL-XTAL X1
+L chiavi-rescue:XTAL-XTAL-teclas-rescue X1
 U 1 1 5EBA8FFC
 P 4200 3100
